Commit message: make hardware_layout also configure the urdf

File: franka_description/robots/sim/dual_panda_arm_sim.urdf.xacro (robot description, xacro)
@@ -7,5 +7,9 @@
   <xacro:arg name="initial_positions_1" default="0.0 ${-pi/4} 0.0 ${-3*pi/4} 0.0 ${pi/2} ${pi/4}"/> <!-- initial joint positions of the robot-->
   <xacro:arg name="initial_positions_2" default="0.0 ${-pi/4} 0.0 ${-3*pi/4} 0.0 ${pi/2} ${pi/4}"/> <!-- initial joint positions of the robot-->
-  <link name="base_link">
+  <xacro:arg name="world_to_base_xyz_1" default="0 0.26 0"/> <!-- world to arm 1 base translation -->
+  <xacro:arg name="world_to_base_rpy_1" default="0 0 0"/> <!-- world to arm 1 base orientation -->
+  <xacro:arg name="world_to_base_xyz_2" default="0 -0.26 0"/> <!-- world to arm 2 base translation -->
+  <xacro:arg name="world_to_base_rpy_2" default="0 0 0"/> <!-- world to arm 2 base orientation -->
+  <link name="world">
     <visual>
       <geometry>
@@ -23,9 +27,9 @@
   <xacro:include filename="$(find franka_description)/robots/common/panda_arm.xacro"/>
   <!--
-  <xacro:panda_arm arm_id="$(arg arm_id_1)" connected_to="base_link" rpy="${-90 * pi/180} 0 ${-90 * pi/180}"  xyz="-143.26e-3 +600e-3 924.51e-3" safety_distance="0.03"/>
-  <xacro:panda_arm arm_id="$(arg arm_id_2)" connected_to="base_link" rpy="${+90 * pi/180} 0 ${+90 * pi/180}"  xyz="-143.26e-3 -600e-3 924.51e-3" safety_distance="0.03"/>
+  <xacro:panda_arm arm_id="$(arg arm_id_1)" connected_to="world" rpy="${-90 * pi/180} 0 ${-90 * pi/180}"  xyz="-143.26e-3 +600e-3 924.51e-3" safety_distance="0.03"/>
+  <xacro:panda_arm arm_id="$(arg arm_id_2)" connected_to="world" rpy="${+90 * pi/180} 0 ${+90 * pi/180}"  xyz="-143.26e-3 -600e-3 924.51e-3" safety_distance="0.03"/>
   -->
-  <xacro:panda_arm arm_id="$(arg arm_id_1)" connected_to="base_link" rpy="0 0 0"  xyz="0 +0.26 0" safety_distance="0.03"/>
-  <xacro:panda_arm arm_id="$(arg arm_id_2)" connected_to="base_link" rpy="0 0 0"  xyz="0 -0.26 0" safety_distance="0.03"/>
+  <xacro:panda_arm arm_id="$(arg arm_id_1)" connected_to="world" rpy="$(arg world_to_base_rpy_1)"  xyz="$(arg world_to_base_xyz_1)" safety_distance="0.03"/>
+  <xacro:panda_arm arm_id="$(arg arm_id_2)" connected_to="world" rpy="$(arg world_to_base_rpy_2)"  xyz="$(arg world_to_base_xyz_2)" safety_distance="0.03"/>
   <xacro:if value="$(arg hand_1)">
     <xacro:include filename="$(find franka_description)/robots/common/hand.xacro"/>
