Commit message: simplify the code to use common

File: franka_description/robots/real/dual_panda_arm.urdf.xacro (robot description, xacro)
@@ -9,5 +9,9 @@
   <xacro:arg name="use_fake_hardware" default="false"/>
   <xacro:arg name="fake_sensor_commands" default="false"/>
-  <link name="base_link">
+  <xacro:arg name="world_to_base_xyz_1" default="0 0.26 0"/> <!-- world to arm 1 base translation -->
+  <xacro:arg name="world_to_base_rpy_1" default="0 0 0"/> <!-- world to arm 1 base orientation -->
+  <xacro:arg name="world_to_base_xyz_2" default="0 -0.26 0"/> <!-- world to arm 2 base translation -->
+  <xacro:arg name="world_to_base_rpy_2" default="0 0 0"/> <!-- world to arm 2 base orientation -->
+  <link name="world">
     <visual>
       <geometry>
@@ -25,9 +29,9 @@
   <xacro:include filename="$(find franka_description)/robots/common/panda_arm.xacro"/>
   <!--
-  <xacro:panda_arm arm_id="$(arg arm_id_1)" connected_to="base_link" rpy="${-90 * pi/180} 0 ${-90 * pi/180}"  xyz="-143.26e-3 +600e-3 924.51e-3" safety_distance="0.03"/>
-  <xacro:panda_arm arm_id="$(arg arm_id_2)" connected_to="base_link" rpy="${+90 * pi/180} 0 ${+90 * pi/180}"  xyz="-143.26e-3 -600e-3 924.51e-3" safety_distance="0.03"/>
+  <xacro:panda_arm arm_id="$(arg arm_id_1)" connected_to="world" rpy="${-90 * pi/180} 0 ${-90 * pi/180}"  xyz="-143.26e-3 +600e-3 924.51e-3" safety_distance="0.03"/>
+  <xacro:panda_arm arm_id="$(arg arm_id_2)" connected_to="world" rpy="${+90 * pi/180} 0 ${+90 * pi/180}"  xyz="-143.26e-3 -600e-3 924.51e-3" safety_distance="0.03"/>
   -->
-  <xacro:panda_arm arm_id="$(arg arm_id_1)" connected_to="base_link" rpy="0 0 0"  xyz="0 +0.26 0" safety_distance="0.03"/>
-  <xacro:panda_arm arm_id="$(arg arm_id_2)" connected_to="base_link" rpy="0 0 0"  xyz="0 -0.26 0" safety_distance="0.03"/>
+  <xacro:panda_arm arm_id="$(arg arm_id_1)" connected_to="world" rpy="$(arg world_to_base_rpy_1)"  xyz="$(arg world_to_base_xyz_1)" safety_distance="0.03"/>
+  <xacro:panda_arm arm_id="$(arg arm_id_2)" connected_to="world" rpy="$(arg world_to_base_rpy_2)"  xyz="$(arg world_to_base_xyz_2)" safety_distance="0.03"/>
   <xacro:if value="$(arg hand_1)">
     <xacro:include filename="$(find franka_description)/robots/common/hand.xacro"/>

File: franka_description/robots/real/panda_arm.urdf.xacro (robot description, xacro)
@@ -6,6 +6,22 @@
   <xacro:arg name="use_fake_hardware" default="false"/>
   <xacro:arg name="fake_sensor_commands" default="false"/>
+  <xacro:arg name="world_to_base_xyz" default="0 0 0"/> <!-- world to base translation -->
+  <xacro:arg name="world_to_base_rpy" default="0 0 0"/> <!-- world to base orientation -->
+  <link name="world">
+    <visual>
+      <geometry>
+         <box size="0.1 0.1 0.1"/>
+      </geometry>
+      <origin rpy="0 0 0" xyz="0 0 0"/>
+    </visual>
+    <collision>
+      <geometry>
+         <box size="0.1 0.1 0.1"/>
+      </geometry>
+      <origin rpy="0 0 0" xyz="0 0 0"/>
+    </collision>
+  </link>
   <xacro:include filename="$(find franka_description)/robots/common/panda_arm.xacro"/>
-  <xacro:panda_arm arm_id="$(arg arm_id)" safety_distance="0.03"/>
+  <xacro:panda_arm arm_id="$(arg arm_id)" connected_to="world" rpy="$(arg world_to_base_rpy)" xyz="$(arg world_to_base_xyz)" safety_distance="0.03"/>
   <xacro:if value="$(arg hand)">
     <xacro:include filename="$(find franka_description)/robots/common/hand.xacro"/>

File: franka_description/robots/sim/panda_arm_sim.urdf.xacro (robot description, xacro)
@@ -4,6 +4,22 @@
   <xacro:arg name="hand" default="true"/> <!-- Should a franka_gripper be mounted at the flange?" -->
   <xacro:arg name="initial_positions" default="0.0 ${-pi/4} 0.0 ${-3*pi/4} 0.0 ${pi/2} ${pi/4}"/> <!-- initial joint positions of the robot-->
+  <xacro:arg name="world_to_base_xyz" default="0 0 0"/> <!-- world to base translation -->
+  <xacro:arg name="world_to_base_rpy" default="0 0 0"/> <!-- world to base orientation -->
+  <link name="world">
+    <visual>
+      <geometry>
+         <box size="0.1 0.1 0.1"/>
+      </geometry>
+      <origin rpy="0 0 0" xyz="0 0 0"/>
+    </visual>
+    <collision>
+      <geometry>
+         <box size="0.1 0.1 0.1"/>
+      </geometry>
+      <origin rpy="0 0 0" xyz="0 0 0"/>
+    </collision>
+  </link>
   <xacro:include filename="$(find franka_description)/robots/common/panda_arm.xacro"/>
-  <xacro:panda_arm arm_id="$(arg arm_id)" safety_distance="0.03"/>
+  <xacro:panda_arm arm_id="$(arg arm_id)" connected_to="world" rpy="$(arg world_to_base_rpy)" xyz="$(arg world_to_base_xyz)" safety_distance="0.03"/>
   <xacro:if value="$(arg hand)">
     <xacro:include filename="$(find franka_description)/robots/common/hand.xacro"/>
